Commit message: fix carpetas

File: src/puzzlebot_description/urdf/model.urdf (robot description, URDF)
Before this commit: robot puzzlebot, 7 links, 6 joints
Links:
- link chassis: geometry collision mesh filename=package://puzzlebot_description/meshes/chassis.stl; visual mesh filename=package://puzzlebot_description/meshes/chassis.stl
- link left_wheel: geometry collision mesh filename=package://puzzlebot_description/meshes/wheel.stl; visual mesh filename=package://puzzlebot_description/meshes/wheel.stl
- link lidar_link: geometry collision mesh filename=package://puzzlebot_description/meshes/LiDAR.stl scale=0.001 0.001 0.001; visual mesh filename=package://puzzlebot_description/meshes/LiDAR.stl scale=0.001 0.001 0.001
- link right_wheel: geometry collision mesh filename=package://puzzlebot_description/meshes/wheel.stl; visual mesh filename=package://puzzlebot_description/meshes/wheel.stl

File: src/puzzlebot_description/urdf/puzzlebot.urdf (robot description, URDF)
Before this commit: robot puzzlebot, 5 links, 4 joints
Links:
- link base_link: geometry visual mesh filename=package://puzzlebot_description/meshes/MCR2_puzzlebot_jetso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
- link caster_link: geometry visual mesh filename=package://puzzlebot_description/meshes/MCR2_caster_wheel.stl
- link wheel_l_link: geometry visual mesh filename=package://puzzlebot_description/meshes/MCR2_wheel.stl
- link wheel_r_link: geometry visual mesh filename=package://puzzlebot_description/meshes/MCR2_wheel.stl
