Commit message: implementacion gazebo

File: src/puzzlebot_description/models/urdf/puzzlebot.urdf (robot description, URDF)
Before this commit: robot puzzlebot, 5 links, 4 joints
Links:
- link base_link: geometry visual mesh filename=package://puzzlebot_description/models/meshes/MCR2_puzzlebo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
- link caster_link: geometry visual mesh filename=package://puzzlebot_description/models/meshes/MCR2_caster_w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
- link wheel_l_link: geometry visual mesh filename=package://puzzlebot_description/models/meshes/MCR2_wheel.stl
- link wheel_r_link: geometry visual mesh filename=package://puzzlebot_description/models/meshes/MCR2_wheel.stl
